File: hardware/KiCad/bmc-lite-hat.kicad_pcb (KiCad board)
At the start: 2 copper layers, 0 parts

Commit message: Update KiCad from Haruna
Parts:
- added REF**: PinHeader_2x20_P2.54mm_Vertical, Connector_PinHeader_2.54mm:PinHeader_2x20_P2.54mm_Vertical, F.Cu at (193.0, 45.7)
- added REF**: XIAO-RP2040-DIP, Seeed Studio XIAO Series Library:XIAO-RP2040-DIP, F.Cu at (177.8, 53.3)

Commit message: Update KiCad from Haruna
Parts:
- added REF**: PinHeader_1x07_P2.54mm_Vertical, Connector_PinHeader_2.54mm:PinHeader_1x07_P2.54mm_Vertical, F.Cu at (185.4, 45.7)
- added REF**: PinHeader_1x07_P2.54mm_Vertical, Connector_PinHeader_2.54mm:PinHeader_1x07_P2.54mm_Vertical, F.Cu at (170.2, 45.7)
- moved REF** 30.5 mm to (147.3, 53.3)
