File: hardware/KiCad/bmc-lite-hat.kicad_sch (KiCad schematic)
At the start: 0 parts

Commit message: Update KiCad from Haruna
Parts:
- added C1: 22 microF, symbol Device:C
- added D1: BAT54CW, Package_TO_SOT_SMD:SOT-323_SC-70, symbol Diode:BAT54CW
- added J1: Conn_02x20_Odd_Even, symbol Connector_Generic:Conn_02x20_Odd_Even
- added U1: XIAO-RP2040-DIP, Module:MOUDLE14P-XIAO-DIP-SMD, symbol Seeed_Studio_XIAO_Series:XIAO-RP2040-DIP
- added U2: MCP23008-xSS, Package_SO:SSOP-20_5.3x7.2mm_P0.65mm, symbol Interface_Expansion:MCP23008-xSS
Connections:
- new net EXP_INT: U1.1 (GPIO26/ADC0/A0), U2.8 (INT)
- new net GND: C1.1, U1.13 (GND)
- new net RPI_UART_RX: U1.7 (GPIO0/TX)
- new net RPI_UART_TX: J1.8 (Pin_8), U1.8 (GPIO1/RX)
- new net SCL: U1.6 (GPIO7/SCL), U2.1 (SCL)
- new net SDA: U1.5 (GPIO6/SDA), U2.2 (SDA)
- new net V_RPI: D1.2, J1.1 (Pin_1)
- new net V_SYS: C1.2, D1.3
- new net V_XIAO: D1.1, U1.12 (3V3)

Commit message: Update KiCad from Haruna
Connections:
- net GND: now also U2.9 (VSS)
- net V_SYS: now also U2.20 (VDD)
Changed lines of the file:
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@@
+		)
+	)
+	(global_label "V_SYS"
+		(shape input)
+		(at 106.68 67.31 90)
+		(fields_autoplaced yes)
+		(effects
+			(font
+				(size 1.27 1.27)
+			)
+			(justify left)
+		)
+		(property "Intersheetrefs" "${INTERSHEET_REFS}"
+			(at 106.68 59.4152 90)
+			(effects
+				(font
+					(size 1.27 1.27)
+				)
+				(justify left)
+				(hide yes)
+			)
 		)
 	)
 	(symbol
 		(lib_id "power:GND")
+		(at 106.68 97.79 0)
+		(unit 1)
+		(exclude_from_sim no)
+		(in_bom yes)
+		(on_board yes)
+		(dnp no)
+		(fields_autoplaced yes)
+		(property "Reference" "#PWR03"
+			(at 106.68 104.14 0)
+			(effects
+				(font
+					(size 1.27 1.27)
+				)
+				(hide yes)
+			)
+		)
+		(property "Value" "GND"
+			(at 106.68 102.87 0)
+			(effects
+				(font
+					(size 1.27 1.27)
+				)
+			)
+		)
+		(property "Footprint" ""
+			(at 106.68 97.79 0)
+			(effects
+				(font
+					(size 1.27 1.27)
+				)
+				(hide yes)
+			)
+		)
+		(property "Datasheet" ""
+			(at 106.68 97.79 0)
+			(effects
+				(font
+					(size 1.27 1.27)
+				)
+				(hide yes)
+			)
+		)
+		(property "Description" "Power symbol creates a global label with name \"GND\" , ground"
+			(at 106.68 97.79 0)
+			(effects
+				(font
+					(size 1.27 1.27)
+				)
+				(hide yes)
+			)
+		)
+		(pin "1"
+		)
+		(instances
+			(project "bmc-lite-hat"
+				(path "/11111111-1111-1111-1111-111111111111"
+					(reference "#PWR03")
+					(unit 1)
+				)
+			)
+		)
+	)
+	(symbol
+		(lib_id "power:GND")

Commit message: Update KiCad from Haruna
Parts:
- removed C1: 22 microF, symbol Device:C
- removed D1: BAT54CW, Package_TO_SOT_SMD:SOT-323_SC-70, symbol Diode:BAT54CW
- added SW2: DEV - RUN POWER ISOLATION, symbol Switch:SW_SPST
Connections:
- net V_SYS is gone; now on net V_XIAO: U2.20 (VDD)
- net GND: now also J1.6 (Pin_6)
- net RPI_UART_RX: now also J1.10 (Pin_10)
- net SHUTDOWN: now reaches J1.11 (Pin_11)
- net REBOOT: now reaches J1.13 (Pin_13)
- net RDY_SHUTDOWN: now reaches J1.29 (Pin_29)
- net HEARTBEAT: now reaches J1.31 (Pin_31)

Commit message: Update KiCad from Haruna
Parts:
- added D1: 1N5819, Diode_THT:D_DO-41_SOD81_P10.16mm_Horizontal, symbol Diode:1N5819
Connections:
- net REBOOT is gone; now on net REBOOT_SIGNAL: J1.13 (Pin_13)
- net SHUTDOWN is gone; now on net SHUTDOWN_SIGNAL: J1.11 (Pin_11)
- net HEARTBEAT: now also U2.19 (GP7)
- net RDY_SHUTDOWN: now also U2.18 (GP6)
- net USER1_SIGNAL: now reaches J1.15 (Pin_15)
- net USER1_SIGNAL: now also U2.16 (GP4)
- net V_RPI_5V: now reaches J1.2 (Pin_2)
- net V_RPI_5V: now also D1.2 (A)
- net V_XIAO_5V: now reaches U1.14 (VBUS)
- net V_XIAO_5V: now also SW2.1 (A)
- net SHUTDOWN_SIGNAL: now reaches U2.12 (GP0)
- net SHUTDOWN_BUTTON: now reaches U2.13 (GP1)
- net REBOOT_SIGNAL: now reaches U2.14 (GP2)
- net REBOOT_BUTTON: now reaches U2.15 (GP3)
- net USER1_BUTTON: now reaches U2.17 (GP5)
- net at SW2.2 (B): now also D1.1 (K)
- net SCL renamed SCL_XIAO
- net SDA renamed SDA_XIAO
- net V_RPI: no longer names the net of J1.1 (Pin_1)
- net V_XIAO renamed V_XIAO_3V3
Other:
- moved on the sheet: SW2, U2
