File: hardware/KiCad/bmc-lite-hat.kicad_sch (KiCad schematic)
At the start: 5 parts, among them J1 Conn_02x20_Odd_Even, SW2 DEV - RUN POWER ISOLATION, U1 XIAO-RP2040-DIP, U2 MCP23008-xSS

Commit message: Update KiCad from Haruna
Other:
- note added: "I2C Expander"
- note added: "RPI GPIO HEADER"
Changed lines of the file:
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@@
 		(comment 1 "Teslamax")
+	)
+	(text "I2C Expander"
+		(exclude_from_sim yes)
+		(at 58.166 105.156 0)
+		(effects
+			(font
+				(size 1.27 1.27)
+			)
+			(justify left)
+		)
+	)
+	(text "RPI GPIO HEADER"
+		(exclude_from_sim yes)
+		(at 220.98 66.548 0)
+		(effects
+			(font
+				(size 1.27 1.27)
+			)
+		)
 	)
 	(wire
