File: hardware/KiCad/bmc-lite-hat.kicad_sch (KiCad schematic)
At the start: 5 parts, among them J1 Conn_02x20_Odd_Even, SW2 DEV - RUN POWER ISOLATION, U1 XIAO-RP2040-DIP, U2 MCP23008-xSS

Commit message: Update KiCad from Haruna
Parts:
- SW1_XIAO-POWER-ISOLATION: renamed from SW2; value DEV - RUN POWER ISOLATION -> DEV - RUN
Changed lines of the file:
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@@
 		(on_board yes)
 		(dnp no)
-		(property "Reference" "SW2"
+		(property "Reference" "SW1_XIAO-POWER-ISOLATION"
 			(at 127 27.94 0)
 			(effects
@@
 			)
 		)
-		(property "Value" "DEV - RUN POWER ISOLATION"
+		(property "Value" "DEV - RUN"
 			(at 127 30.48 0)
 			(effects
@@
 			(project ""
 				(path "/11111111-1111-1111-1111-111111111111"
-					(reference "SW2")
+					(reference "SW1_XIAO-POWER-ISOLATION")
 					(unit 1)
 				)

Commit message: Update hardware files
Parts:
- added U3: MCP23017_SP, Package_DIP:DIP-28_W7.62mm, symbol Interface_Expansion:MCP23017_SP
Connections:
- net EXP_INT: now also U3.20 (INTA)
- net GND: now also U3.10 (VSS)
- net HEARTBEAT: now also U3.28 (GPA7)
- net RDY_SHUTDOWN: now also U3.27 (GPA6)
- net REBOOT_BUTTON: now also U3.24 (GPA3)
- net REBOOT_SIGNAL: now also U3.23 (GPA2)
- net SCL_XIAO: now also U3.12 (SCK)
- net SDA_XIAO: now also U3.13 (SDA)
- net SHUTDOWN_BUTTON: now also U3.22 (GPA1)
- net SHUTDOWN_SIGNAL: now also U3.21 (GPA0)
- net USER1_BUTTON: now also U3.26 (GPA5)
- net USER1_SIGNAL: now also U3.25 (GPA4)
- net V_XIAO_3V3: now also U3.9 (VDD)
Other:
- moved on the sheet: U2
